File: keeb_mini.kicad_pcb (KiCad board)
At the start: 2 copper layers, 67 parts, among them J2 Conn_01x02, SW1 SW_Push, SW10 SW_Push, SW11 SW_Push, SW12 SW_Push, SW13 SW_Push, SW14 SW_Push, SW15 SW_Push, SW16 SW_Push, SW17 SW_Push, SW18 SW_Push, SW19 SW_Push, SW2 SW_Push, SW20 SW_Push, SW21 SW_Push, SW22 SW_Push, SW23 SW_Push, SW24 SW_Push, SW25 SW_Push, SW26 SW_Push, SW27 SW_Push, SW28 SW_Push, SW29 SW_Push, SW3 SW_Push, SW30 SW_Push, SW4 SW_Push, SW5 SW_Push, SW6 SW_Push, SW7 SW_Push, SW8 SW_Push, SW9 SW_Push, U1 NCP1117-3.3_SOT223, U2 RP2040, U3 W25Q128JVS

Commit message: Started PCB making, encountered issues with routing
Parts:
- added C1: 100nF, Capacitor_SMD:C_0805_2012Metric, F.Cu at (79.0, 153.4)
- added C10: 100nF, Capacitor_SMD:C_0805_2012Metric, F.Cu at (62.3, 139.5)
- added C11: 100nF, Capacitor_SMD:C_0805_2012Metric, F.Cu at (51.2, 151.7)
- added C13: 27pF, Capacitor_SMD:C_0805_2012Metric, F.Cu at (96.3, 164.8)
- added C14: 27pF, Capacitor_SMD:C_0805_2012Metric, F.Cu at (96.3, 156.3)
- added C15: 10uF, Capacitor_SMD:C_0805_2012Metric, F.Cu at (1.73, 1.00)
- added C16: 10uF, Capacitor_SMD:C_0805_2012Metric, F.Cu at (1.73, 4.01)
- added C2: 100nF, Capacitor_SMD:C_0805_2012Metric, F.Cu at (51.1, 158.2)
- added C3: 100nF, Capacitor_SMD:C_0805_2012Metric, F.Cu at (64.6, 166.1)
- added C4: 100nF, Capacitor_SMD:C_0805_2012Metric, F.Cu at (68.2, 166.0)
- added C5: 100nF, Capacitor_SMD:C_0805_2012Metric, F.Cu at (78.9, 156.4)
- added C6: 100nF, Capacitor_SMD:C_0805_2012Metric, F.Cu at (68.3, 143.5)
- added C7: 100nF, Capacitor_SMD:C_0805_2012Metric, F.Cu at (64.6, 143.4)
- added C8: 100nF, Capacitor_SMD:C_0805_2012Metric, F.Cu at (51.0, 155.0)
- added C9: 1uF, Capacitor_SMD:C_0805_2012Metric, F.Cu at (60.2, 143.9)
- added J1: USB4110GFA, Connector_USB:USB_C_Receptacle_GCT_USB4110, F.Cu at (166.6, 22.2)
- added R1: 5k1, Resistor_SMD:R_0805_2012Metric, F.Cu at (16.4, 16.0)
- added R2: 5k1, Resistor_SMD:R_0805_2012Metric, F.Cu at (16.4, 19.0)
- added R3: 27k, Resistor_SMD:R_0805_2012Metric, F.Cu at (56.1, 149.2)
- added R4: 27k, Resistor_SMD:R_0805_2012Metric, F.Cu at (56.1, 146.2)
- added R6: 1k, Resistor_SMD:R_0805_2012Metric, F.Cu at (78.6, 159.7)
- added Y1: ABLS-12.000MHZ-B4-T, Crystal:Crystal_SMD_HC49-SD, F.Cu at (88.7, 160.6)
- C12: value 100n -> 100nF; footprint Capacitor_SMD:C_0402_1005Metric -> Capacitor_SMD:C_0805_2012Metric
- D1, D10, D11, D12, D13, D14, D15, D16, D17, D18, D19, D2, D20, D21, D22, D23, D24, D25, D26, D27, D28, D29, D3, D30, D4, D5, D6, D7, D8, D9: footprint Diode_THT:D_DO-35_SOD27_P7.62mm_Horizontal -> Diode_SMD:D_SOD-523
- R5, R7: footprint Resistor_SMD:R_0402_1005Metric -> Resistor_SMD:R_0805_2012Metric
- moved SW21 177.2 mm to (72.4, 99.8)
- moved SW22 152.1 mm to (91.4, 99.8)
- moved U3 140.9 mm to (47.7, 167.5), turned to 90 degrees
- moved SW11 132.6 mm to (72.4, 80.7)
- moved D10 128.3 mm to (240.0, 66.7), turned to 90 degrees
- moved SW23 128.0 mm to (110.5, 99.8)
- moved U2 114.7 mm to (67.3, 155.2), turned to 90 degrees
- moved SW26 112.6 mm to (167.6, 99.8)
- moved D9 112.4 mm to (221.0, 66.6), turned to 90 degrees
- moved SW12 107.7 mm to (91.4, 80.7)
- moved SW24 105.8 mm to (129.5, 99.8)
- moved D20 105.5 mm to (240.0, 85.7), turned to 90 degrees
- moved D11 104.8 mm to (68.6, 85.7), turned to 90 degrees
- moved D21 100.3 mm to (68.6, 104.8), turned to 90 degrees
- moved D8 97.6 mm to (201.9, 66.7), turned to 90 degrees
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Connections:
- U2 pad 11: unconnected-(U2-GPIO8-Pad11) -> /COL8
- U2 pad 12: unconnected-(U2-GPIO9-Pad12) -> /COL9
- U2 pad 15: unconnected-(U2-GPIO12-Pad15) -> /ROW0
- U2 pad 16: unconnected-(U2-GPIO13-Pad16) -> /ROW1
- U2 pad 17: unconnected-(U2-GPIO14-Pad17) -> /ROW2
- U2 pad 2: unconnected-(U2-GPIO0-Pad2) -> /COL0
- U2 pad 3: unconnected-(U2-GPIO1-Pad3) -> /COL1
- U2 pad 4: unconnected-(U2-GPIO2-Pad4) -> /COL2
- U2 pad 5: unconnected-(U2-GPIO3-Pad5) -> /COL3
- U2 pad 6: unconnected-(U2-GPIO4-Pad6) -> /COL4
- U2 pad 7: unconnected-(U2-GPIO5-Pad7) -> /COL5
- U2 pad 8: unconnected-(U2-GPIO6-Pad8) -> /COL6
- U2 pad 9: unconnected-(U2-GPIO7-Pad9) -> /COL7
Routing:
- net /ROW2: track 0.00 -> 171.5 mm
- net /ROW1: track 0.00 -> 171.4 mm
- net /ROW0: track 0.00 -> 171.4 mm
- net Net-(U2-ADC_AVDD): track 0.00 -> 81.9 mm
- net /COL9: track 0.00 -> 38.1 mm
- net /COL8: track 0.00 -> 38.1 mm
- net /COL7: track 0.00 -> 38.1 mm
- net /COL6: track 0.00 -> 38.1 mm
- net /COL5: track 0.00 -> 38.1 mm
- net /COL4: track 0.00 -> 38.1 mm
- net /COL3: track 0.00 -> 38.1 mm
- net /COL2: track 0.00 -> 38.1 mm
- net /COL1: track 0.00 -> 38.1 mm
- net /COL0: track 0.00 -> 38.1 mm
- net /XIN: track 0.00 -> 29.2 mm
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